File: file55EF2C93.sch (KiCad schematic (older format))
At the start: 17 parts, among them U11 4000series-4052, U12 4000series-4052, U13 4000series-4052

Commit message: more work on the clock schematic. Almost done!
Parts:
- added C1, C?: 10n, symbol C_Small
- added C6: 22000uF, symbol CP_Small
- added D? (x2): D, symbol D
- added P?: USB_B, symbol USB_B
- added Q? (x8): 2N7000, symbol 2N7000
- added R1, R? (x3): 22K, symbol R
- added R25: 100R, symbol R
- added R? (x8): 82R, symbol R
- added SW?: HOUR, symbol SW_PUSH_SMALL
- added SW?: MIN, symbol SW_PUSH_SMALL
- added SW?: SET, symbol SW_PUSH_SMALL
- added SW?: RUN, symbol SW_PUSH_SMALL
- added U1: 4000series-4093, symbol 4000series-4093
- added U7: 4000series-4081, symbol 4000series-4081
- added U8: 4000series-4543, symbol 4000series-4543
Connections:
- net +5V: now also C6.1, D?.1 (K), R1.1, R?.1, R?.1, R?.1, U8.1 (LD)
- net +5VD: now also D?.1 (K)
- net A: now also R?.1
- net B: now also R?.1
- net C: now also R?.1
- net D: now also R?.1
- net E: now also R?.1
- net F: now also R?.1
- net G: now also R?.1
- net GND: now also C1.2, C?.2, P?.4 (GND), P?.5 (shield), Q?.1 (S), Q?.1 (S), Q?.1 (S), Q?.1 (S), Q?.1 (S), Q?.1 (S), Q?.1 (S), Q?.1 (S), R25.2, SW?.1, SW?.1, SW?.1, SW?.1, U8.6 (PH)
- net MIN0: now also U11.12 (X0)
- net MIN1: now also U11.1 (Y0)
- net MIN4: now also U11.14 (X1)
- net MIN5: now also U11.5 (Y1)
- net MSD: now also U7.13
- net DP: now reaches 7SEG?.9 (DP2)
- net DP: now also 7SEG?.9 (DP2), R?.1
- net sC: now reaches U12.13 (X_COM)
- net sC: now also U8.2 (sC)
- net sD: now reaches U12.3 (Y_COM)
- net sD: now also U8.4 (sD)
- net HR4: now reaches U11.11 (X3)
- net sA: now reaches U11.13 (X_COM)
- net sA: now also U8.5 (sA)
- net HR0: now reaches U11.15 (X2)
- net HR1: now reaches U11.2 (Y2)
- net sB: now reaches U11.3 (Y_COM)
- net sB: now also U8.3 (sB)
- net HR5: now reaches U11.4 (Y3)
- new net: Q?.2 (G), U8.10 (B)
- new net: Q?.2 (G), U8.11 (C)
- new net: Q?.2 (G), U8.12 (D)
- new net: Q?.2 (G), U8.13 (E)
- new net: Q?.2 (G), U8.14 (G)
- new net: Q?.2 (G), U8.15 (F)
- new net: U7.11, U8.7 (BI)
- new net: Q?.2 (G), U8.9 (A)
- new net: C?.1, R?.2, SW?.2, U1.8, U1.9
- new net: R?.2, SW?.2, U1.12, U1.13
- new net: Q?.3 (D), R?.2 (x8)
- new net: Q?.2 (G), U7.10
- new net: D?.2 (A), D?.2 (A), P?.1 (VCC)
- new net: C6.2, R25.1
- new net: C1.1, R1.2, SW?.2, U1.1
- new net: R?.2, SW?.2, U1.6
- new net 0.5HZ: U7.8
- new net HOUR: U1.10
- new net LEAD0: U7.12
- new net MIN: U1.11
- new net SET: U1.3, U1.5
- new net ~SET: U1.2, U1.4, U7.9
- no-connect marks 0 -> 4
Other:
- note added: "Digital Design of CMOS-CLOCK by\nSan Bergmans of sbprojects.com"
- moved on the sheet: 7SEG?, Q?, R?
