File: file55EF2C93.sch (KiCad schematic (older format))
At the start: 51 parts, among them U1 4000series-4093, U11 4000series-4052, U12 4000series-4052, U13 4000series-4052, U7 4000series-4081, U8 4000series-4543

Commit message: More work on the clock
Parts:
- removed 7SEG? (x2): OSL20561-IX, symbol OSL20561-IX
- removed Q? (x4): BC327-25, TO-92, symbol BC327-25
- removed R?: 100K, symbol R
- removed R?: 2K2, symbol R
- added 7SEG? (x4): SC08-11EWA, symbol SC08-11EWA
- added Q?: 2N7002, symbol 2N7002
- added R?: 100K, symbol R
Connections:
- wire segments 213 -> 214
- no-connect marks 4 -> 5
Other:
- note added: "Min Digits are mounted upside\ndown for use of DP as seconds\nSo connections get swapped\naround"
- note removed: "Digit is mounted upside down\nfor use of DP as middle colon.\nSo connections get swapped\naround"
- moved on the sheet: R?, U11A, U12A, U13A

Commit message: Added common cathode displays and other stuff
Parts:
- removed R? (x3): 100K, symbol R
- removed R? (x3): 2K2, symbol R
- removed U8: 4000series-4543, symbol 4000series-4543
- added C?: 10pF, symbol C
- added C?: 39pF, symbol CTRIM
- added Q? (x3): 2N7002, symbol 2N7002
- added R? (x7): 100K, symbol R
- added R?: 10M, symbol R
- added R?: 220K, symbol R
- added TP?: 32768Hz, symbol CONN_01X01
- added U?: 4000series-4060, symbol 4000series-4060
- added U?: 4000series-4511, symbol 4000series-4511
- added Y?: 32768Hz, symbol Crystal
- renumbered C6 to C?, C1 to C?, R25 to R?, R1 to R?, U13 to U?, U12 to U?, U11 to U?, U1 to U?, U7 to U?
Connections:
- net labels removed: DIG1, DIG2
- wire segments 214 -> 217
Other:
- note added: "TIMEBASE"
- note removed: "Digital Design of CMOS-CLOCK by\nSan Bergmans of sbprojects.com"
- note removed: "Min Digits are mounted upside\ndown for use of DP as seconds\nSo connections get swapped\naround"
- moved on the sheet: 7SEG?, Q?, R?, U?A

Commit message: Changing to a single 4-digit common anode display
Parts:
- removed 7SEG? (x4): SC08-11EWA, symbol SC08-11EWA
- removed Q? (x4): 2N7002, symbol 2N7002
- removed R? (x8): 100K, symbol R
- added 7SEG?: CA56-21, symbol CA56-21
- added Q?: 2N7000, symbol 2N7000
Connections:
- net labels added: DIG1, DIG2
- wire segments 217 -> 167
- no-connect marks 5 -> 2
Other:
- note added: "DISPLAY"
- moved on the sheet: Q?, R?, U?A

Commit message: More work on the CMOS clock
Parts:
- added U?: 4000series-4013, symbol 4000series-4013
- R?: value 10M -> 15M
Connections:
- net GND: now also U?.4 (R), U?.6 (S)
- net 64Hz: now reaches U?.13 (Q9)
- net 128Hz: now reaches U?.14 (Q8)
- net at U?.3 (Q14): now also U?.3
- new net: U?.2 (~Q), U?.5 (D)
- new net 1Hz: U?.1 (Q)
